File: hw/IO_module.brd (EAGLE design)
At the start: 25 x 45 mm, 22 parts, among them J1 R2P_BUS-VERTICAL, J2 R2P_BUS-VERTICAL

Commit message: Layout complete
Parts:
- added RN1, RN2, RN3, RN4, RN5: 220, r2p_rcl:RNET4_1206
- added RN6: (no value), r2p_rcl:RNET4_1206
- added U$10, U$11, U$12, U$13: MOLEX_53047-06, r2p_connector:MOLEX_53047-06
- added X1, X2, X3, X4: MOLEX_53047-04, r2p_connector:MOLEX_53047-04
- moved C14 0.50 mm to (9.50, 21.4)
Connections:
- new net ADC2_IN12: RN5.1, U$6.20
- new net ADC2_IN3: RN5.4, U$6.16
- new net ADC2_IN4: RN5.3, U$6.17
- new net ADC3_IN1: RN5.2, U$6.19
- new net DAC_OUT1: RN6.3, U$6.14, X4.3
- new net DAC_OUT2: RN6.4, U$6.15, X4.4
- new net I2C2_SCL: RN6.1, U$6.30, X1.3
- new net I2C2_SDA: RN6.2, U$6.31, X1.4
- new net N$11: RN1.6, X3.4
- new net N$12: RN2.8, U$10.6
- new net N$13: RN2.7, U$10.5
- new net N$14: RN2.6, U$10.4
- new net N$15: RN2.5, U$10.3
- new net N$18: RN5.8, U$13.6
- new net N$19: RN5.7, U$13.5
- new net N$20: RN5.6, U$13.4
- new net N$21: RN5.5, U$13.3
- new net N$22: RN4.5, U$12.3
- new net N$23: RN4.6, U$12.4
- new net N$24: RN4.7, U$12.5
- new net N$25: RN4.8, U$12.6
- new net N$26: RN3.5, U$11.3
- new net N$27: RN3.6, U$11.4
- new net N$28: RN3.7, U$11.5
- new net N$29: RN3.8, U$11.6
- new net N$3: RN1.5, X3.3
- new net N$5: RN1.7, X2.3
- new net N$6: RN1.8, X2.4
- new net SPI2_MISO: RN2.2, U$6.27
- new net SPI2_MOSI: RN2.1, U$6.28
- new net SPI2_NSS: RN2.4, U$6.25
- new net SPI2_SCK: RN2.3, U$6.26
- new net TIM1_CH1: RN4.1, U$6.29
- new net TIM2_CH1: RN3.4, U$6.10
- new net TIM2_CH2: RN3.3, U$6.11
- new net TIM2_CH3: RN3.2, U$6.12
- new net TIM2_CH4: RN3.1, U$6.13
- new net TIM3_CH1: RN4.4, U$6.40
- new net TIM3_CH2: RN4.3, U$6.41
- new net TIM3_CH3: RN4.2, U$6.18
- new net UART1_RX: RN1.1, U$6.43
- new net UART1_TX: RN1.2, U$6.42
- new net UART3_RX: RN1.3, U$6.22
- new net UART3_TX: RN1.4, U$6.21
- new net USB_DM: U$6.32
- new net USB_DP: U$6.33
- net +3V3: now also RN6.7, RN6.8, U$10.1, U$11.1, U$12.1, U$13.1, X1.1, X2.1, X3.1, X4.1
- net GND: now also RN6.5, RN6.6, U$10.2, U$11.2, U$12.2, U$13.2, X1.2, X2.2, X3.2, X4.2
Routing:
- net +3V3: track 78.8 -> 151.8 mm, vias 7 -> 8
- net DAC_OUT1: track 0.00 -> 43.6 mm, vias 0 -> 2
- net DAC_OUT2: track 0.00 -> 42.9 mm, vias 0 -> 2
- net UART1_RX: track 0.00 -> 22.7 mm, vias 0 -> 2
- net UART1_TX: track 0.00 -> 22.6 mm, vias 0 -> 2
- net N$21: track 0.00 -> 20.0 mm
- net I2C2_SDA: track 0.00 -> 19.3 mm
- net N$20: track 0.00 -> 19.1 mm
- net N$29: track 0.00 -> 18.7 mm
- net N$19: track 0.00 -> 18.2 mm
- net I2C2_SCL: track 0.00 -> 18.1 mm
- net N$28: track 0.00 -> 17.8 mm
- net N$18: track 0.00 -> 17.1 mm
- net N$27: track 0.00 -> 16.9 mm
- net TIM3_CH1: track 0.00 -> 16.7 mm, vias 0 -> 2
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Other:
- board text added: "ADC"
- board text added: "D1"
- board text added: "D2"
- board text added: "DAC"
- board text added: "I2C"
- board text added: "IO module v1.0 (2014/02)"
- board text added: "SPI"
- board text added: "UART 1"
- board text added: "UART 2"
- board text removed: "R2P module v0.0 (YYYY/MM)"

Commit message: Updated keepout
Parts:
- U$2: value LPS4018 -> (none)
Changed lines of the file:
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@@
 <attribute name="VALUE" x="20.905" y="3.2" size="0.635" layer="27" font="vector" ratio="10" rot="R180"/>
 </element>
-<element name="U$2" library="r2p_rcl" package="COILCRAFT_LPS4018" value="LPS4018" x="11.2" y="8.7" smashed="yes" rot="R90"/>
+<element name="U$2" library="r2p_rcl" package="COILCRAFT_LPS4018" value="" x="11.2" y="8.7" smashed="yes" rot="R90"/>
 <element name="C1" library="r2p_rcl" package="C1206" value="1u" x="4.1" y="8.9" smashed="yes" rot="R90">
 <attribute name="NAME" x="4.1" y="8.9" size="1" layer="25" font="vector" rot="R90" align="center"/>
