File: hw/IO_module.sch (EAGLE design)
At the start: 22 parts, among them J1 R2P_BUS-VERTICAL, J2 R2P_BUS-VERTICAL

Commit message: Layout complete
Parts:
- added RN1, RN2, RN3, RN4, RN5: 220, r2p_rcl:RNETWORK_4-1206
- added RN6: (no value), r2p_rcl:RNETWORK_4-1206
- added U$10, U$11, U$12, U$13: MOLEX_53047-06, r2p_connector:MOLEX_53047-06
- added X1, X2, X3, X4: MOLEX_53047-04, r2p_connector:MOLEX_53047-04
Connections:
- new net ADC2_IN12: RN5G$1.1, U$6.PB2-BOOT1
- new net ADC2_IN3: RN5G$4.1, U$6.PA6
- new net ADC2_IN4: RN5G$3.1, U$6.PA7
- new net ADC3_IN1: RN5G$2.1, U$6.PB1
- new net DAC_OUT1: RN6G$3.1, U$6.PA4, X43.S
- new net DAC_OUT2: RN6G$4.1, U$6.PA5, X44.S
- new net I2C2_SCL: RN6G$1.1, U$6.PA9, X13.S
- new net I2C2_SDA: RN6G$2.1, U$6.PA10, X14.S
- new net N$11: RN1G$3.2, X34.S
- new net N$12: RN2G$1.2, U$106.S
- new net N$13: RN2G$2.2, U$105.S
- new net N$14: RN2G$3.2, U$104.S
- new net N$15: RN2G$4.2, U$103.S
- new net N$18: RN5G$1.2, U$136.S
- new net N$19: RN5G$2.2, U$135.S
- new net N$20: RN5G$3.2, U$134.S
- new net N$21: RN5G$4.2, U$133.S
- new net N$22: RN4G$4.2, U$123.S
- new net N$23: RN4G$3.2, U$124.S
- new net N$24: RN4G$2.2, U$125.S
- new net N$25: RN4G$1.2, U$126.S
- new net N$26: RN3G$4.2, U$113.S
- new net N$27: RN3G$3.2, U$114.S
- new net N$28: RN3G$2.2, U$115.S
- new net N$29: RN3G$1.2, U$116.S
- new net N$3: RN1G$4.2, X33.S
- new net N$5: RN1G$2.2, X23.S
- new net N$6: RN1G$1.2, X24.S
- new net SPI2_MISO: RN2G$2.1, U$6.PB14
- new net SPI2_MOSI: RN2G$1.1, U$6.PB15
- new net SPI2_NSS: RN2G$4.1, U$6.PB12
- new net SPI2_SCK: RN2G$3.1, U$6.PB13
- new net TIM1_CH1: RN4G$1.1, U$6.PA8
- new net TIM2_CH1: RN3G$4.1, U$6.PA0/WKUP
- new net TIM2_CH2: RN3G$3.1, U$6.PA1
- new net TIM2_CH3: RN3G$2.1, U$6.PA2
- new net TIM2_CH4: RN3G$1.1, U$6.PA3
- new net TIM3_CH1: RN4G$4.1, U$6.PB4
- new net TIM3_CH2: RN4G$3.1, U$6.PB5
- new net TIM3_CH3: RN4G$2.1, U$6.PB0
- new net UART1_RX: RN1G$1.1, U$6.PB7
- new net UART1_TX: RN1G$2.1, U$6.PB6
- new net UART3_RX: RN1G$3.1, U$6.PB11
- new net UART3_TX: RN1G$4.1, U$6.PB10
- new net USB_DM: U$6.PA11
- new net USB_DP: U$6.PA12
- net +3V3: now also RN6G$1.2, RN6G$2.2, U$101.S, U$111.S, U$121.S, U$131.S, X11.S, X21.S, X31.S, X41.S
- net GND: now also RN6G$3.2, RN6G$4.2, U$102.S, U$112.S, U$122.S, U$132.S, X12.S, X22.S, X32.S, X42.S

Commit message: Updated keepout
Parts:
- C1: device r2p_rcl:C-1206 -> r2p_rcl:C1206
- C14, C17, C2, C3, C4, C6, C7, C8: device r2p_rcl:C-0603 -> r2p_rcl:C0603
- C5, C9: device r2p_rcl:C-0805 -> r2p_rcl:C0805
- R1: device r2p_rcl:R-0603 -> r2p_rcl:R0603
- U$2: value LPS4018 -> (none)
Changed lines of the file:
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@@
 </classes>
 <parts>
-<part name="C6" library="r2p_rcl" deviceset="C" device="-0603" value="10n"/>
+<part name="C6" library="r2p_rcl" deviceset="C" device="0603" value="10n"/>
 <part name="GND11" library="r2p_supply" deviceset="GND" device=""/>
 <part name="GND12" library="r2p_supply" deviceset="GND" device=""/>
@@
 <part name="GND6" library="r2p_supply" deviceset="GND" device=""/>
 <part name="+3V4" library="r2p_supply" deviceset="+3V3" device=""/>
-<part name="C17" library="r2p_rcl" deviceset="C" device="-0603" value="100n"/>
-<part name="C14" library="r2p_rcl" deviceset="C" device="-0603" value="100n"/>
-<part name="C4" library="r2p_rcl" deviceset="C" device="-0603" value="100n"/>
+<part name="C17" library="r2p_rcl" deviceset="C" device="0603" value="100n"/>
+<part name="C14" library="r2p_rcl" deviceset="C" device="0603" value="100n"/>
+<part name="C4" library="r2p_rcl" deviceset="C" device="0603" value="100n"/>
 <part name="GND29" library="r2p_supply" deviceset="GND" device=""/>
 <part name="GND30" library="r2p_supply" deviceset="GND" device=""/>
 <part name="GND31" library="r2p_supply" deviceset="GND" device=""/>
 <part name="+3V11" library="r2p_supply" deviceset="+3V3" device=""/>
-<part name="C5" library="r2p_rcl" deviceset="C" device="-0805" value="4.7u"/>
+<part name="C5" library="r2p_rcl" deviceset="C" device="0805" value="4.7u"/>
 <part name="GND34" library="r2p_supply" deviceset="GND" device=""/>
 <part name="+3V5" library="r2p_supply" deviceset="+3V3" device=""/>
 <part name="GND7" library="r2p_supply" deviceset="GND" device=""/>
 <part name="+3V6" library="r2p_supply" deviceset="+3V3" device=""/>
-<part name="C3" library="r2p_rcl" deviceset="C" device="-0603" value="100n"/>
+<part name="C3" library="r2p_rcl" deviceset="C" device="0603" value="100n"/>
 <part name="GND9" library="r2p_supply" deviceset="GND" device=""/>
 <part name="+3V3" library="r2p_supply" deviceset="+3V3" device=""/>
 <part name="GND8" library="r2p_supply" deviceset="GND" device=""/>
 <part name="GND10" library="r2p_supply" deviceset="GND" device=""/>
-<part name="C7" library="r2p_rcl" deviceset="C" device="-0603" value="100n"/>
+<part name="C7" library="r2p_rcl" deviceset="C" device="0603" value="100n"/>
 <part name="GND22" library="r2p_supply" deviceset="GND" device=""/>
 <part name="LED1" library="r2p_led" deviceset="LED" device="0805" value=""/>
-<part name="R1" library="r2p_rcl" deviceset="R" device="-0603" value="330"/>
+<part name="R1" library="r2p_rcl" deviceset="R" device="0603" value="330"/>
 <part name="GND16" library="r2p_supply" deviceset="GND" device=""/>
 <part name="GND17" library="r2p_supply" deviceset="GND" device=""/>
@@
 <part name="J2" library="r2p_connector" deviceset="R2P_BUS" device="-VERTICAL"/>
 <part name="U$2" library="r2p_rcl" deviceset="LPS4018" device=""/>
-<part name="C1" library="r2p_rcl" deviceset="C" device="-1206" value="1u"/>
+<part name="C1" library="r2p_rcl" deviceset="C" device="1206" value="1u"/>
 <part name="GND1" library="r2p_supply" deviceset="GND" device=""/>
-<part name="C2" library="r2p_rcl" deviceset="C" device="-0603" value="1u"/>
-<part name="C8" library="r2p_rcl" deviceset="C" device="-0603" value="10n"/>
+<part name="C2" library="r2p_rcl" deviceset="C" device="0603" value="1u"/>
+<part name="C8" library="r2p_rcl" deviceset="C" device="0603" value="10n"/>
 <part name="GND4" library="r2p_supply" deviceset="GND" device=""/>
 <part name="GND5" library="r2p_supply" deviceset="GND" device=""/>
-<part name="C9" library="r2p_rcl" deviceset="C" device="-0805" value="10u"/>
+<part name="C9" library="r2p_rcl" deviceset="C" device="0805" value="10u"/>
 <part name="GND2" library="r2p_supply" deviceset="GND" device=""/>
 <part name="GND3" library="r2p_supply" deviceset="GND" device=""/>
